File: Firefly5/Firefly5_hw/Firefly5.kicad_pcb (KiCad board)
At the start: 2 copper layers, 57 x 12 mm, 31 parts, among them Q1 ALS, Q2 LED_RGB 5050, SW1 SWITCH

Commit message: Layout done
Parts:
- removed D2: LED, LED-3MM
- removed F1: FUSE0R, SMD0603_FUSE
- removed XL2: ST_SWD, SIL-4
- removed XL3: CONN_1, SIL1_SQUARE_1MM5
- removed XL4, XL6: CONN_1, SIL1_ROUND_1MM5
- removed XL5: CONN_8, SIL-8
- added ANT1: ANT_GENERAL, Radio:ANT_2400_MEANDER_MIRR, F.Cu at (220.0, 98.9)
- added B1: BAT, Installation:BATTERY_AA, B.Cu at (191.0, 103.1)
- added C11: 0.1u, Capacitors:CAP_0603, F.Cu at (165.2, 109.3)
- added C12: 18pF, Capacitors:CAP_0603, F.Cu at (202.7, 109.2)
- added C13: 1u, Capacitors:CAP_0603, F.Cu at (203.2, 97.0)
- added C14: 18pF, Capacitors:CAP_0603, F.Cu at (208.9, 109.2)
- added C15: 220pF, Capacitors:CAP_0603, F.Cu at (208.0, 97.0)
- added C16: 0.1u, Capacitors:CAP_0603, F.Cu at (200.9, 104.2)
- added C17: 0.1u, Capacitors:CAP_0603, F.Cu at (210.4, 98.1)
- added C18: 0.1u, Capacitors:CAP_0603, F.Cu at (210.4, 106.1)
- added C19: 220pF, Capacitors:CAP_0603, F.Cu at (205.7, 106.4)
- added C20: 0.1u, Capacitors:CAP_0603, F.Cu at (200.9, 102.6)
- added C21: 220pF, Capacitors:CAP_0603, F.Cu at (204.8, 97.0)
- added C22: 100pF, Capacitors:CAP_0402, F.Cu at (210.3, 103.7)
- added C23: 100pF, Capacitors:CAP_0402, F.Cu at (210.3, 101.3)
- added C24: 1pF, Capacitors:CAP_0402, F.Cu at (212.0, 104.2)
- added C25: 1pF, Capacitors:CAP_0402, F.Cu at (213.7, 101.3)
- added C26: 1.8pF, Capacitors:CAP_0402, F.Cu at (214.2, 99.6)
- added C27: 1.5pF, Capacitors:CAP_0402, F.Cu at (215.4, 104.2)
- added DD2: CC2500, QFN_DFN:QFN20, F.Cu at (205.9, 102.3)
- added L2: 1.2nH, Inductors:IND_0402, F.Cu at (212.0, 100.8)
- added L3: 1.2nH, Inductors:IND_0402, F.Cu at (213.7, 103.7)
- added L4: 1.2nH, Inductors:IND_0402, F.Cu at (214.9, 102.5)
- added R6: 56k, Resistors:RES_0603, F.Cu at (198.9, 110.1)
- added R7: 56k, Resistors:RES_0603, F.Cu at (206.4, 97.0)
- added SW2: Btn4x4, BtnsSwitches:BTN_4x4_SMD, F.Cu at (173.1, 107.9)
- added SW3: Btn4x4, BtnsSwitches:BTN_4x4_SMD, F.Cu at (173.1, 98.3)
- added XTAL1: 27MHz, Quartz:03225C4, F.Cu at (205.8, 109.2)
- C1: value 0.1u -> 10u; footprint CAP_0603 -> Capacitors:CAP_0603
- C10: value 1u -> 0.1u; footprint CAP_0603 -> Capacitors:CAP_0603
- C2, C3, C4, C8: footprint CAP_0603 -> Capacitors:CAP_0603
- C5: value 0.1u -> 10n; footprint CAP_0603 -> Capacitors:CAP_0603
- C6: value 0.1u -> 1u; footprint CAP_0603 -> Capacitors:CAP_0603
- C7, C9: footprint CAP_0805 -> Capacitors:CAP_0603
- D1: value BAT54WS -> PMEG2020; footprint DIODE_SOD323 -> Diodes:SOD323
- DA1: footprint SOT23-5 -> SOT:SOT23-5
- DD1: value STM32F100C4 -> STM32F030C8Tx; footprint LQFP48 -> LQFP_TQFP:LQFP48
- L1: footprint IND_1210 -> Inductors:IND_1210_LQH32C
- Q1: value ALS -> LED_5050; footprint RES_0603 -> LEDs:LED_5050
- Q2: value LED_RGB 5050 -> ALS-PT19-315C; footprint LED_HH5050_RGB -> Resistors:RES_0603
- R1, R3, R5: footprint RES_0603 -> Resistors:RES_0603
- R2: value 10k -> 51R; footprint RES_0603 -> Resistors:RES_0603
- R4: value 51R -> 10k; footprint RES_0603 -> Resistors:RES_0603
- SW1: footprint SIL-3 -> BtnsSwitches:SW_SS-1P2T
- TP1: footprint TESTPOINT_0_5MM -> PCB:TESTPOINT_1MM
- XL1: value CONN_3 -> CONN_6; footprint SIL-3 -> Connectors:PLS-6
- moved Q1 100.2 mm to (196.2, 103.1)
- moved C6 94.9 mm to (194.7, 108.5)
- moved C1 81.1 mm to (179.4, 99.6)
- moved R2 80.6 mm to (196.3, 97.6), turned to 270 degrees
- moved XL1 80.0 mm to (191.0, 96.6)
- moved C3 76.7 mm to (191.5, 98.7), turned to 0 degrees
- moved DA1 75.5 mm to (179.7, 107.0), turned to 0 degrees
- moved TP1 74.4 mm to (200.4, 107.6)
- moved D1 73.8 mm to (180.9, 102.7)
- moved L1 73.1 mm to (178.0, 103.1)
- moved SW1 71.4 mm to (170.1, 103.1)
- moved C9 70.1 mm to (180.4, 110.1), turned to 0 degrees
- moved C5 67.4 mm to (194.7, 110.1)
- moved R1 66.9 mm to (197.9, 97.6), turned to 270 degrees
- moved C7 66.6 mm to (167.3, 100.1), turned to 180 degrees
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Connections:
- C1 pad 1: N-000007 -> +3.3V
- C6 pad 1: +BATT -> +3.3V
- C8 pad 1: +3.3V -> +BATT
- DD1 pad 10: (no net) -> /BTN1
- DD1 pad 11: N-0000028 -> /LUM_MEAS
- DD1 pad 12: N-0000027 -> Net-(DD1-Pad12)
- DD1 pad 13: N-0000020 -> /CC_GDO0
- DD1 pad 14: /5 -> /CC_CS
- DD1 pad 15: /6 -> /CC_SCK
- DD1 pad 16: /7 -> /CC_MISO
- DD1 pad 17: /8 -> /CC_MOSI
- DD1 pad 18: N-000004 -> /RED_LED
- DD1 pad 19: N-000007 -> /GREEN_LED
- DD1 pad 2: (no net) -> /BTN2
- DD1 pad 30: /TX -> /UART_TX
- DD1 pad 31: /RX -> /UART_RX
- DD1 pad 34: /SB_SWDAT -> /SWDIO
- DD1 pad 35: GND -> (no net)
- DD1 pad 36: +3.3V -> (no net)
- DD1 pad 37: /SB_SWCLK -> /SWCLK
- DD1 pad 39: /4 -> (no net)
- DD1 pad 40: (no net) -> /BLUE_LED
- DD1 pad 42: /3 -> (no net)
- DD1 pad 43: /2 -> (no net)
- DD1 pad 7: N-000006 -> (no net)
- Q1 pad 1: +3.3V -> Net-(Q1-Pad1)
- Q1 pad 2: N-000007 -> Net-(Q1-Pad2)
- R1 pad 1: N-0000027 -> /BLUE_LED
- R1 pad 2: N-0000029 -> Net-(Q1-Pad1)
- R2 pad 1: +BATT -> /RED_LED
- R2 pad 2: N-000004 -> Net-(Q1-Pad2)
- R3 pad 1: N-0000020 -> /GREEN_LED
- R3 pad 2: N-0000030 -> Net-(Q1-Pad3)
- R4 pad 1: N-0000028 -> +BATT
- R4 pad 2: N-000008 -> Net-(DD1-Pad12)
- R5 pad 1: N-000007 -> /LUM_MEAS
- TP1 pad 1: N-000006 -> /CC_GDO0
- XL1 pad 1: /RX -> +3.3V
- XL1 pad 2: /TX -> /SWCLK
Routing:
- net GND: track 173.2 -> 0.00 mm, vias 23 -> 0
- net +3.3V: track 72.9 -> 0.00 mm, vias 5 -> 0
- net N-000007: track 31.3 -> 0.00 mm, vias 2 -> 0
- net /8: track 29.6 -> 0.00 mm
- net +BATT: track 27.5 -> 0.00 mm
- net /7: track 27.3 -> 0.00 mm
- net /6: track 25.4 -> 0.00 mm
- net /4: track 24.5 -> 0.00 mm, vias 1 -> 0
- net /5: track 24.3 -> 0.00 mm
- net /3: track 20.8 -> 0.00 mm, vias 1 -> 0
- net /2: track 17.6 -> 0.00 mm, vias 1 -> 0
- net /TX: track 12.7 -> 0.00 mm, vias 1 -> 0
- net /SB_SWCLK: track 12.4 -> 0.00 mm, vias 1 -> 0
- net /RX: track 10.1 -> 0.00 mm, vias 1 -> 0
- net N-000004: track 9.99 -> 0.00 mm, vias 2 -> 0
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- removed copper zone on B.Cu, net GND
- removed copper zone on F.Cu, net GND
Other:
- board size 57 x 12 mm -> 63 x 16 mm
- net class Default: clearance 0.2 -> 0
- rule trace_clearance: 0.2 -> 0

Commit message: Firefly5 ready for production
Parts:
- added Logo1: Logo, Pictures:Ostranna_8x8, F.Cu at (221.8, 99.9)
- moved C19 0.41 mm to (205.6, 106.0)
- moved ANT1 0.30 mm to (220.0, 98.6)
- moved R1 0.22 mm to (197.8, 97.8)
- moved R2 0.22 mm to (196.2, 97.8)
- moved R3 0.22 mm to (194.6, 97.8)
Connections:
- DA1 pad 3: (no net) -> Net-(DA1-Pad3)
- DD1 pad 20: (no net) -> Net-(DD1-Pad20)
- DD1 pad 21: (no net) -> Net-(DD1-Pad21)
- DD1 pad 22: (no net) -> Net-(DD1-Pad22)
- DD1 pad 25: (no net) -> Net-(DD1-Pad25)
- DD1 pad 26: (no net) -> Net-(DD1-Pad26)
- DD1 pad 27: (no net) -> Net-(DD1-Pad27)
- DD1 pad 28: (no net) -> Net-(DD1-Pad28)
- DD1 pad 29: (no net) -> Net-(DD1-Pad29)
- DD1 pad 3: (no net) -> Net-(DD1-Pad3)
- DD1 pad 32: (no net) -> Net-(DD1-Pad32)
- DD1 pad 33: (no net) -> Net-(DD1-Pad33)
- DD1 pad 35: (no net) -> Net-(DD1-Pad35)
- DD1 pad 36: (no net) -> Net-(DD1-Pad36)
- DD1 pad 38: (no net) -> Net-(DD1-Pad38)
- DD1 pad 39: (no net) -> Net-(DD1-Pad39)
- DD1 pad 4: (no net) -> Net-(DD1-Pad4)
- DD1 pad 41: (no net) -> Net-(DD1-Pad41)
- DD1 pad 42: (no net) -> Net-(DD1-Pad42)
- DD1 pad 43: (no net) -> Net-(DD1-Pad43)
- DD1 pad 45: (no net) -> Net-(DD1-Pad45)
- DD1 pad 46: (no net) -> Net-(DD1-Pad46)
- DD1 pad 5: (no net) -> Net-(DD1-Pad5)
- DD1 pad 6: (no net) -> Net-(DD1-Pad6)
- DD1 pad 7: (no net) -> Net-(DD1-Pad7)
- DD2 pad 3: (no net) -> Net-(DD2-Pad3)
- SW1 pad 3: (no net) -> Net-(SW1-Pad3)
Routing:
- net GND: track 0.00 -> 249.7 mm, vias 0 -> 58
- net +3.3V: track 0.00 -> 150.7 mm, vias 0 -> 10
- net /BTN2: track 0.00 -> 32.3 mm, vias 0 -> 2
- net Net-(DD1-Pad12): track 0.00 -> 32.0 mm, vias 0 -> 2
- net /LUM_MEAS: track 0.00 -> 29.8 mm, vias 0 -> 2
- net /BTN1: track 0.00 -> 22.8 mm, vias 0 -> 2
- net /CC_CS: track 0.00 -> 19.9 mm, vias 0 -> 2
- net /BLUE_LED: track 0.00 -> 18.8 mm, vias 0 -> 2
- net /CC_MISO: track 0.00 -> 15.6 mm
- net /CC_GDO0: track 0.00 -> 15.3 mm, vias 0 -> 2
- net /CC_MOSI: track 0.00 -> 14.8 mm
- net +BATT: track 0.00 -> 14.6 mm
- net /CC_SCK: track 0.00 -> 13.1 mm
- net /SWCLK: track 0.00 -> 10.9 mm, vias 0 -> 1
- net Net-(ANT1-Pad1): track 0.00 -> 10.6 mm
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- added copper zone on B.Cu, net GND
- added copper zone on F.Cu, net GND
Other:
- net class Default: trace_width 0.2 -> 0.18; via_dia 0.9 -> 0.7; via_drill 0.4 -> 0.3
- net class Wide: clearance 0.2 -> 0.18
- rule trace_min: 0.2 -> 0.1
- rule via_min_drill: 0.4 -> 0.3
- rule via_min_size: 0.889 -> 0.6
- board text added: "Ostranna Firefly5"

Commit message: * Something in FF3 + FF5.1
Parts:
- D1: value PMEG2020 -> BAT60
- Q2: value ALS-PT19-315C -> TEMT7000X01; footprint Resistors:RES_0603 -> Resistors:RES_0805
- R1, R2, R3: value 51R -> 100R
- moved Logo1 54.1 mm to (196.3, 147.6), turned to 180 degrees
- moved ANT1 52.2 mm to (197.6, 145.8), turned to 0 degrees
- moved C26 44.1 mm to (196.6, 140.0), turned to 180 degrees
- moved C27 43.8 mm to (192.0, 141.2), turned to 0 degrees
- moved L4 43.7 mm to (193.7, 140.7), turned to 90 degrees
- moved C25 42.6 mm to (194.9, 139.5), turned to 270 degrees
- moved L3 41.6 mm to (192.5, 139.5), turned to 90 degrees
- moved L2 40.6 mm to (195.4, 137.8), turned to 0 degrees
- moved C17 40.0 mm to (198.1, 136.2), turned to 0 degrees
- moved C24 39.1 mm to (192.0, 137.8), turned to 0 degrees
- moved C23 38.1 mm to (194.9, 136.1), turned to 270 degrees
- moved C15 37.8 mm to (199.2, 133.8), turned to 0 degrees
- moved C22 37.0 mm to (192.5, 136.1), turned to 270 degrees
- moved C18 36.3 mm to (190.1, 136.2), turned to 270 degrees
- moved R7 35.9 mm to (199.2, 132.2), turned to 0 degrees
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Connections:
- DA1 pad 3: Net-(DA1-Pad3) -> (no net)
- DD1 pad 20: Net-(DD1-Pad20) -> (no net)
- DD1 pad 21: Net-(DD1-Pad21) -> (no net)
- DD1 pad 22: Net-(DD1-Pad22) -> (no net)
- DD1 pad 25: Net-(DD1-Pad25) -> (no net)
- DD1 pad 26: Net-(DD1-Pad26) -> (no net)
- DD1 pad 27: Net-(DD1-Pad27) -> (no net)
- DD1 pad 28: Net-(DD1-Pad28) -> (no net)
- DD1 pad 3: Net-(DD1-Pad3) -> (no net)
- DD1 pad 32: Net-(DD1-Pad32) -> (no net)
- DD1 pad 33: Net-(DD1-Pad33) -> (no net)
- DD1 pad 35: Net-(DD1-Pad35) -> (no net)
- DD1 pad 36: Net-(DD1-Pad36) -> (no net)
- DD1 pad 38: Net-(DD1-Pad38) -> (no net)
- DD1 pad 39: Net-(DD1-Pad39) -> (no net)
- DD1 pad 4: Net-(DD1-Pad4) -> (no net)
- DD1 pad 41: Net-(DD1-Pad41) -> (no net)
- DD1 pad 42: Net-(DD1-Pad42) -> (no net)
- DD1 pad 43: Net-(DD1-Pad43) -> (no net)
- DD1 pad 45: Net-(DD1-Pad45) -> (no net)
- DD1 pad 46: Net-(DD1-Pad46) -> (no net)
- DD1 pad 5: Net-(DD1-Pad5) -> (no net)
- DD1 pad 6: Net-(DD1-Pad6) -> (no net)
- DD1 pad 7: Net-(DD1-Pad7) -> (no net)
- DD2 pad 3: Net-(DD2-Pad3) -> (no net)
- Q2 pad 1: +3.3V -> /LUM_MEAS
- Q2 pad 2: /LUM_MEAS -> GND
- R5 pad 1: /LUM_MEAS -> Net-(DD1-Pad29)
- R5 pad 2: GND -> /LUM_MEAS
- SW1 pad 3: Net-(SW1-Pad3) -> (no net)
Routing:
- net GND: track 249.7 -> 156.6 mm, vias 58 -> 27
- net /BTN2: track 32.3 -> 122.2 mm, vias 2 -> 25
- net /Lout: track 4.81 -> 66.6 mm, vias 0 -> 4
- net Net-(DD1-Pad12): track 32.0 -> 0.00 mm, vias 2 -> 0
- net /LUM_MEAS: track 29.8 -> 0.00 mm, vias 2 -> 0
- net /BTN1: track 22.8 -> 0.00 mm, vias 2 -> 0
- net Net-(DD1-Pad21): track 0.00 -> 22.3 mm, vias 0 -> 2
- net Net-(SW1-Pad3): track 0.00 -> 21.5 mm, vias 0 -> 9
- net /CC_GDO0: track 15.3 -> 0.00 mm, vias 2 -> 0
- net /SWCLK: track 10.9 -> 0.00 mm, vias 1 -> 0
- net /CC_SCK: track 13.1 -> 3.08 mm
- net +3.3V: track 150.7 -> 159.4 mm, vias 10 -> 12
- net /RED_LED: track 8.69 -> 0.00 mm, vias 2 -> 0
- net /SWDIO: track 8.02 -> 0.00 mm, vias 1 -> 0
- net Net-(DD1-Pad45): track 0.00 -> 6.39 mm
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Other:
- board size 63 x 16 mm -> 16 x 63 mm
- net class Default: trace_width 0.18 -> 0.25
- board text added: "E"

Commit message: Firefly 5.1 sent to factory
Parts:
- DD1: value STM32F030C8Tx -> STM32F030C8T6
- moved R4 73.9 mm to (147.9, 146.2), turned to 270 degrees
- moved Logo1 72.4 mm to (150.5, 91.5), turned to 0 degrees
- moved C8 71.8 mm to (149.5, 146.2), turned to 270 degrees
- moved ANT1 71.0 mm to (149.6, 93.5), turned to 180 degrees
- moved C7 69.6 mm to (151.1, 146.2), turned to 270 degrees
- moved Q2 66.1 mm to (159.9, 149.8), turned to 180 degrees
- moved SW3 63.9 mm to (149.3, 140.4), turned to 270 degrees
- moved C11 62.5 mm to (160.3, 147.9), turned to 180 degrees
- moved C26 61.4 mm to (150.6, 99.3), turned to 0 degrees
- moved SW1 61.3 mm to (154.1, 143.3), turned to 90 degrees
- moved R5 59.6 mm to (160.3, 146.3), turned to 180 degrees
- moved C17 59.1 mm to (149.1, 103.2), turned to 180 degrees
- moved C15 58.5 mm to (148.0, 105.5), turned to 180 degrees
- moved C25 58.2 mm to (152.3, 99.8), turned to 90 degrees
- moved L4 58.2 mm to (153.5, 98.7), turned to 270 degrees
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Routing:
- net /BTN2: track 122.2 -> 32.2 mm, vias 25 -> 2
- net GND: track 156.6 -> 236.5 mm, vias 27 -> 58
- net /Lout: track 66.6 -> 4.81 mm, vias 4 -> 0
- net Net-(DD1-Pad12): track 0.00 -> 32.2 mm, vias 0 -> 2
- net /LUM_MEAS: track 0.00 -> 30.2 mm, vias 0 -> 2
- net /BTN1: track 0.00 -> 22.9 mm, vias 0 -> 2
- net Net-(DD1-Pad21): track 22.3 -> 0.00 mm, vias 2 -> 0
- net Net-(DD1-Pad29): track 0.00 -> 22.1 mm, vias 0 -> 2
- net Net-(SW1-Pad3): track 21.5 -> 0.00 mm, vias 9 -> 0
- net +3.3V: track 159.4 -> 141.3 mm, vias 12 -> 10
- net /CC_GDO0: track 0.00 -> 15.2 mm, vias 0 -> 2
- net /SWCLK: track 0.00 -> 10.9 mm, vias 0 -> 1
- net /CC_SCK: track 3.08 -> 13.4 mm
- net /RED_LED: track 0.00 -> 8.69 mm, vias 0 -> 2
- net /SWDIO: track 0.00 -> 6.57 mm, vias 0 -> 1
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Other:
- board text added: "Ostranna Firefly5.1"
- board text removed: "Ostranna Firefly5"
